File: hardware/recur_control.kicad_pcb (KiCad board)
At the start: 2 copper layers, 100 x 100 mm, 45 parts, among them J1 mono_jack_3.5mm, J2 mono_jack_3.5mm, J3 mono_jack_3.5mm, J4 mono_jack_3.5mm, SW1 Push, SW10 Push, SW11 Push, SW12 Push, SW13 Push, SW14 Push, SW15 Push, SW16 Push, SW17 Push, SW18 Push, SW19 Push, SW2 Push, SW20 Push, SW3 Push, SW4 Push, SW5 Push, SW6 Push, SW7 Push, SW8 Push, SW9 Push, U1 ProMicro

Commit message: update code and circuit revision
Parts:
- J1, J2, J3, J4: footprint Connector_Audio:Jack_3.5mm_QingPu_WQP-PJ398SM_Vertical_CircularHoles -> lib_fp:Jack_3.5mm_QingPu_WQP-PJ398SM_Vertical_CircularHoles
- RV1, RV2, RV3, RV4: footprint Potentiometer_THT:Potentiometer_Alps_RK09L_Single_Vertical -> lib_fp:Potentiometer_Alps_RK09L_Single_Vertical
- U1: footprint project_parts:ProMicro -> lib_fp:ProMicro
Other:
- board text added: "c_l_i_k_r v0_2_1 cyberboy666"
- board text removed: "c_l_i_k_r v0_2 cyberboy666"
